File: full adder.kicad_sch (KiCad schematic)
At the start: 53 parts, among them J1 Barrel_Jack

Commit message: commit
Parts:
- added SW1, SW2, SW3, SW4: SW_SPDT, symbol Switch:SW_SPDT

Commit message: commmit
Parts:
- removed SW1, SW2, SW3, SW4: SW_SPDT, symbol Switch:SW_SPDT
- added SW5, SW6: SW_SPDT, symbol Switch:SW_SPDT
Connections:
- net GND: now also SW5.1 (A), SW6.1 (A)

Commit message: COMMIT
Parts:
- added D17, D18, D19, D20, D21, D22, D23, D24: LED, symbol Device:LED
- added R33, R34, R35, R36, R37, R38, R39, R40: 1K, symbol Device:R
- added SW1, SW10, SW11, SW12, SW13, SW14, SW15, SW16, SW2, SW3, SW4, SW7, SW8, SW9: SW_SPDT, symbol Switch:SW_SPDT
Connections:
- net A0: now also R1.2, R2.1, SW3.2 (B)
- net A1: now also R3.2, R4.1, SW5.2 (B)
- net A2: now also R5.2, R6.1, SW1.2 (B)
- net A3: now also R7.2, R8.1, SW2.2 (B)
- net A4: now also R10.1, R9.2, SW4.2 (B)
- net A5: now also R11.2, R12.1, SW6.2 (B)
- net A6: now also R13.2, R14.1, SW7.2 (B)
- net A7: now also R15.2, R16.1, SW8.2 (B)
- net GND: now also D17.1 (K), D18.1 (K), D19.1 (K), D20.1 (K), D21.1 (K), D22.1 (K), D23.1 (K), D24.1 (K), SW1.1 (A), SW10.1 (A), SW11.1 (A), SW12.1 (A), SW13.1 (A), SW14.1 (A), SW15.1 (A), SW16.1 (A), SW2.1 (A), SW3.1 (A), SW4.1 (A), SW7.1 (A), SW8.1 (A), SW9.1 (A)
- net SUB: no longer R1.1, R11.1, R13.1, R15.1, R17.1, R19.1, R21.1, R23.1, R25.1, R27.1, R29.1, R3.1, R31.1, R5.1, R7.1, R9.1
- net B4: now reaches R25.2, R26.1
- net B4: now also IC3.12 (A4), SW13.2 (B)
- net B7: now reaches R31.2, R32.1
- net B7: now also IC3.1 (A1), SW16.2 (B)
- net B6: now reaches R29.2, R30.1
- net B6: now also IC3.4 (A2), SW15.2 (B)
- net B2: now reaches R21.2, R22.1
- net B2: now also IC4.4 (A2), SW11.2 (B)
- net B0: now reaches R17.2, R18.1
- net B0: now also IC4.12 (A4), SW9.2 (B)
- net S7: now reaches IC1.15 (S3)
- net S7: now also R33.1
- net S6: now reaches IC1.2 (S2)
- net S6: now also R34.1
- net S5: now reaches IC1.6 (S1)
- net S5: now also R35.1
- net S4: now reaches IC1.9 (S0)
- net S4: now also R36.1
- net B1: now reaches R19.2, R20.1
- net B1: now also IC4.9 (A3), SW10.2 (B)
- net B5: now reaches R27.2, R28.1
- net B5: now also IC3.9 (A3), SW14.2 (B)
- net B3: now reaches R23.2, R24.1
- net B3: now also IC4.1 (A1), SW12.2 (B)
- net S3: now reaches IC2.15 (S3)
- net S3: now also R37.1
- net S2: now reaches IC2.2 (S2)
- net S2: now also R38.1
- net S1: now reaches IC2.6 (S1)
- net S1: now also R39.1
- net S0: now reaches IC2.9 (S0)
- net S0: now also R40.1
- net +5V renamed VCC
- net VCC: now also R1.1, R11.1, R13.1, R15.1, R17.1, R19.1, R21.1, R23.1, R25.1, R27.1, R29.1, R3.1, R31.1, R5.1, R7.1, R9.1
- new net: D24.2 (A), R40.2
- new net: D23.2 (A), R39.2
- new net: D17.2 (A), R33.2
- new net: D21.2 (A), R37.2
- new net: D22.2 (A), R38.2
- new net: D19.2 (A), R35.2
- new net: D20.2 (A), R36.2
- new net: D18.2 (A), R34.2
- no-connect marks 1 -> 17
Other:
- note added: "7483"
- note added: "7486"
- moved on the sheet: IC2, IC4

Commit message: COMMIT
Parts:
- added R41: R, symbol Device:R
- added SW17: SW_Push, symbol Switch:SW_Push
Connections:
- net GND: now also SW17.1
- net SUB: now also R41.2, SW17.2
- net VCC: now also R41.1
Changed lines of the file:
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@@
 	)
 	(junction
+		(at 147.32 152.4)
+		(diameter 0)
+		(color 0 0 0 0)
+	)
+	(junction
 		(at 241.3 96.52)
 		(diameter 0)
@@
 	(wire
 		(pts
+			(xy 142.24 152.4) (xy 147.32 152.4)
+		)
+		(stroke
+			(width 0)
+			(type default)
+		)
+	)
+	(wire
+		(pts
 			(xy 31.75 35.56) (xy 36.83 35.56)
 		)
@@
 		)
 	)
+	(label "VCC"
+		(at 147.32 144.78 0)
+		(effects
+			(font
+				(size 1.27 1.27)
+			)
+			(justify left bottom)
+		)
+	)
 	(label "B7"
 		(at 92.71 44.45 0)
@@
 		)
 	)
+	(label "SUB"
+		(at 142.24 152.4 0)
+		(effects
+			(font
+				(size 1.27 1.27)
+			)
+			(justify left bottom)
+		)
+	)
 	(label "VCC"
 		(at 200.66 55.88 0)
@@
 	)
 	(symbol
+		(lib_id "Device:R")
+		(at 147.32 148.59 0)
+		(unit 1)
+		(exclude_from_sim no)
+		(in_bom yes)
+		(on_board yes)
+		(dnp no)
+		(fields_autoplaced yes)
+		(property "Reference" "R41"
+			(at 149.86 147.3199 0)
+			(effects
+				(font
+					(size 1.27 1.27)
+				)
+				(justify left)
+			)
+		)
+		(property "Value" "R"
+			(at 149.86 149.8599 0)
+			(effects
+				(font
+					(size 1.27 1.27)
+				)
+				(justify left)
+			)
+		)
+		(property "Footprint" ""
+			(at 145.542 148.59 90)
+			(effects
+				(font
+					(size 1.27 1.27)
+				)
+				(hide yes)
+			)
+		)
+		(property "Datasheet" "~"
+			(at 147.32 148.59 0)
+			(effects
+				(font
+					(size 1.27 1.27)
+				)
+				(hide yes)
+			)
+		)
+		(property "Description" "Resistor"
+			(at 147.32 148.59 0)
+			(effects
+				(font
+					(size 1.27 1.27)
+				)
+				(hide yes)
+			)
+		)
+		(pin "2"
+		)
+		(pin "1"
+		)
+		(instances
+			(project ""
+				(path "/3df54633-31c2-4102-8885-9302cfc48dc4"
+					(reference "R41")
+					(unit 1)
+				)
+			)
+		)
+	)
+	(symbol
 		(lib_id "power:GND")
 		(at 265.43 66.04 0)
@@
 	(symbol
 		(lib_id "power:GND")
+		(at 147.32 162.56 0)
+		(unit 1)
+		(exclude_from_sim no)
+		(in_bom yes)
+		(on_board yes)
+		(dnp no)
+		(fields_autoplaced yes)
+		(property "Reference" "#PWR046"
+			(at 147.32 168.91 0)
+			(effects
+				(font
+					(size 1.27 1.27)
+				)
+				(hide yes)
+			)
+		)
+		(property "Value" "GND"
+			(at 147.32 167.64 0)
+			(effects
+				(font
+					(size 1.27 1.27)
+				)
+			)
+		)
+		(property "Footprint" ""
+			(at 147.32 162.56 0)
+			(effects
+				(font
+					(size 1.27 1.27)
+				)
+				(hide yes)
+			)
+		)
+		(property "Datasheet" ""
+			(at 147.32 162.56 0)
+			(effects
+				(font
+					(size 1.27 1.27)
+				)
+				(hide yes)
+			)
+		)
+		(property "Description" "Power symbol creates a global label with name \"GND\" , ground"
+			(at 147.32 162.56 0)
+			(effects
+				(font
+					(size 1.27 1.27)
+				)
+				(hide yes)
+			)
+		)
+		(pin "1"
+		)
+		(instances
+			(project ""
+				(path "/3df54633-31c2-4102-8885-9302cfc48dc4"
+					(reference "#PWR046")
+					(unit 1)
+				)
+			)
+		)
+	)
+	(symbol
+		(lib_id "power:GND")
 		(at 191.77 160.02 0)
 		(unit 1)
@@
 					(unit 1)
 				)
+			)
+		)
+	)
+	(symbol
+		(lib_id "Switch:SW_Push")
+		(at 147.32 157.48 90)
+		(unit 1)
+		(exclude_from_sim no)
+		(in_bom yes)
+		(on_board yes)
+		(dnp no)
+		(fields_autoplaced yes)
+		(property "Reference" "SW17"
+			(at 148.59 156.2099 90)
+			(effects
+				(font
+					(size 1.27 1.27)
+				)
+				(justify right)
+			)
+		)
+		(property "Value" "SW_Push"
+			(at 148.59 158.7499 90)
+			(effects
+				(font
+					(size 1.27 1.27)
+				)
+				(justify right)
+			)
+		)
+		(property "Footprint" ""
+			(at 142.24 157.48 0)
+			(effects
+				(font
+					(size 1.27 1.27)
+				)
+				(hide yes)
+			)
+		)
+		(property "Datasheet" "~"
+			(at 142.24 157.48 0)
+			(effects
+				(font
+					(size 1.27 1.27)
+				)
+				(hide yes)
+			)
+		)
+		(property "Description" "Push button switch, generic, two pins"
+			(at 147.32 157.48 0)
+			(effects
+				(font
+					(size 1.27 1.27)
+				)
+				(hide yes)
+			)
+		)
+		(pin "1"
+		)
+		(pin "2"
+		)
+		(instances
+			(project ""
+				(path "/3df54633-31c2-4102-8885-9302cfc48dc4"
+					(reference "SW17")
+					(unit 1)
+				)

Commit message: commit
Parts:
- D1, D10, D11, D12, D13, D14, D15, D16, D17, D18, D19, D2, D20, D21, D22, D23, D24, D3, D4, D5, D6, D7, D8, D9: footprint (none) -> LED_THT:LED_D3.0mm
- IC1, IC2: footprint (none) -> Package_DIP:DIP-16_W7.62mm
- IC3, IC4: footprint (none) -> Package_DIP:DIP-14_W7.62mm
- R1, R10, R11, R12, R13, R14, R15, R16, R17, R18, R19, R2, R20, R21, R22, R23, R24, R25, R26, R27, R28, R29, R3, R30, R31, R32, R33, R34, R35, R36, R37, R38, R39, R4, R40, R41, R5, R6, R7, R8, R9: footprint (none) -> Resistor_THT:R_Axial_DIN0204_L3.6mm_D1.6mm_P5.08mm_Horizontal

Commit message: co
Parts:
- J1: footprint (none) -> Connector_BarrelJack:BarrelJack_Horizontal
- SW1, SW10, SW11, SW12, SW13, SW14, SW15, SW16, SW2, SW3, SW4, SW5, SW6, SW7, SW8, SW9: footprint (none) -> new switch:new switch
- SW17: footprint (none) -> Button_Switch_THT:SW_PUSH_6mm
Changed lines of the file:
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@@
 			)
 		)
-		(property "Footprint" ""
+		(property "Footprint" "new switch:new switch"
 			(at 100.33 182.88 0)
 			(effects
@@
 			)
 		)
-		(property "Footprint" ""
+		(property "Footprint" "new switch:new switch"
 			(at 79.9318 182.88 0)
 			(effects
@@
 			)
 		)
-		(property "Footprint" ""
+		(property "Footprint" "new switch:new switch"
 			(at 54.61 165.1 0)
 			(effects
@@
 			)
 		)
-		(property "Footprint" ""
+		(property "Footprint" "new switch:new switch"
 			(at 24.13 165.1 0)
 			(effects
@@
 		(on_board yes)
 		(dnp no)
-		(fields_autoplaced yes)
 		(property "Reference" "#PWR01"
 			(at 34.29 46.99 0)
@@
 			)
 		)
-		(property "Footprint" ""
+		(property "Footprint" "Connector_BarrelJack:BarrelJack_Horizontal"
 			(at 25.4 39.116 0)
 			(effects
@@
 			)
 		)
-		(property "Footprint" ""
+		(property "Footprint" "new switch:new switch"
 			(at 85.09 165.1 0)
 			(effects
@@
 		(on_board yes)
 		(dnp no)
-		(fields_autoplaced yes)
 		(property "Reference" "#FLG01"
 			(at 36.83 33.655 0)
@@
 			)
 		)
-		(property "Footprint" ""
+		(property "Footprint" "Button_Switch_THT:SW_PUSH_6mm"
 			(at 142.24 157.48 0)
 			(effects
@@
 			)
 		)
-		(property "Footprint" ""
+		(property "Footprint" "new switch:new switch"
 			(at 39.37 182.88 0)
 			(effects
@@
 			)
 		)
-		(property "Footprint" ""
+		(property "Footprint" "new switch:new switch"
 			(at 69.7718 182.88 0)
 			(effects
@@
 			)
 		)
-		(property "Footprint" ""
+		(property "Footprint" "new switch:new switch"
 			(at 64.6918 165.1 0)
 			(effects
@@
 			)
 		)
-		(property "Footprint" ""
+		(property "Footprint" "new switch:new switch"
 			(at 90.17 182.88 0)
 			(effects
@@
 			)
 		)
-		(property "Footprint" ""
+		(property "Footprint" "new switch:new switch"
 			(at 29.21 182.88 0)
 			(effects
@@
 			)
 		)
-		(property "Footprint" ""
+		(property "Footprint" "new switch:new switch"
 			(at 74.8518 165.1 0)
 			(effects
@@
 			)
 		)
-		(property "Footprint" ""
+		(property "Footprint" "new switch:new switch"
 			(at 49.53 182.88 0)
 			(effects
@@
 			)
 		)
-		(property "Footprint" ""
+		(property "Footprint" "new switch:new switch"
 			(at 34.29 165.1 0)
 			(effects
@@
 			)
 		)
-		(property "Footprint" ""
+		(property "Footprint" "new switch:new switch"
 			(at 95.25 165.1 0)
 			(effects
@@
 			)
 		)
-		(property "Footprint" ""
+		(property "Footprint" "new switch:new switch"
 			(at 59.69 182.88 0)
 			(effects
@@
 			)
 		)
-		(property "Footprint" ""
+		(property "Footprint" "new switch:new switch"
 			(at 44.45 165.1 0)
 			(effects
