File: full adder.kicad_pcb (KiCad board)
At the start: 2 copper layers, 87 parts, among them J1 Barrel_Jack, SW1 SW_SPDT, SW10 SW_SPDT, SW11 SW_SPDT, SW12 SW_SPDT, SW13 SW_SPDT, SW14 SW_SPDT, SW15 SW_SPDT, SW16 SW_SPDT, SW17 SW_Push, SW2 SW_SPDT, SW3 SW_SPDT, SW4 SW_SPDT, SW5 SW_SPDT, SW6 SW_SPDT, SW7 SW_SPDT, SW8 SW_SPDT, SW9 SW_SPDT

Commit message: commit
Parts:
- moved SW16 202.0 mm to (239.0, 163.0)
- moved SW8 197.5 mm to (227.0, 142.0)
- moved SW9 175.5 mm to (71.0, 163.0)
- moved SW7 149.5 mm to (203.0, 142.0)
- moved SW3 138.5 mm to (59.0, 142.0)
- moved SW13 103.8 mm to (167.0, 163.0)
- moved SW6 101.5 mm to (179.0, 142.0)
- moved SW5 90.5 mm to (83.0, 142.0)
- moved SW10 64.2 mm to (95.0, 163.0)
- moved SW4 53.5 mm to (155.0, 142.0)
- moved SW1 42.5 mm to (107.0, 142.0)
- moved SW12 32.8 mm to (143.0, 163.0)
- moved SW15 32.3 mm to (215.0, 163.0)
- moved SW14 16.9 mm to (191.0, 163.0)
- moved SW11 16.0 mm to (119.0, 163.0)
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Routing:
- net /VCC: track 171.1 -> 43.4 mm
- net /A0: track 98.5 -> 8.92 mm
- net /S0: track 73.1 -> 0.00 mm
- net GND: track 111.5 -> 43.5 mm
- net Net-(D16-A): track 12.9 -> 4.42 mm
- net Net-(D14-A): track 12.9 -> 4.46 mm
- net Net-(D13-A): track 12.9 -> 4.46 mm
- net Net-(D12-A): track 12.9 -> 4.42 mm
- net Net-(D15-A): track 13.0 -> 4.54 mm
- net Net-(D11-A): track 13.0 -> 4.95 mm
- net Net-(D10-A): track 12.7 -> 4.85 mm
- net Net-(D9-A): track 13.0 -> 5.28 mm
- net Net-(D2-A): track 12.5 -> 5.00 mm
- net Net-(D4-A): track 12.4 -> 4.96 mm
- net Net-(D3-A): track 12.4 -> 4.96 mm
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
Commit message: commit
Parts:
- removed D17: LED, LED_THT:LED_D3.0mm
- added D25: LED, LED_THT:LED_D3.0mm, F.Cu at (182.5, 46.9)
- IC1, IC2: value ~ -> 7483
- IC3, IC4: value ~ -> 7486
- J1: footprint Connector_BarrelJack:BarrelJack_Horizontal -> Connector_BarrelJack:BarrelJack_GCT_DCJ200-10-A_Horizontal
- R1, R10, R11, R12, R13, R14, R15, R16, R17, R18, R19, R2, R20, R21, R22, R23, R24, R25, R26, R27, R28, R29, R3, R30, R31, R32, R33, R34, R35, R36, R37, R38, R39, R4, R40, R5, R6, R7, R8, R9: value 1K -> 1k
- SW1, SW10, SW11, SW12, SW13, SW14, SW15, SW16, SW2, SW3, SW4, SW5, SW6, SW7, SW8, SW9: footprint new switch:new switch -> my footprtn:LED SWITCH3pin
- moved R33 137.2 mm to (164.2, 27.0)
- moved R34 135.2 mm to (172.5, 35.1)
- moved R35 132.6 mm to (168.2, 27.0)
- moved R36 129.3 mm to (176.2, 35.1)
- moved R37 127.2 mm to (172.3, 27.0)
- moved R38 122.3 mm to (180.2, 35.2)
- moved R39 121.0 mm to (176.1, 27.0)
- moved D20 120.5 mm to (164.3, 46.8)
- moved R40 120.0 mm to (180.2, 27.1)
- moved D18 118.5 mm to (150.8, 46.9)
- moved D19 117.8 mm to (155.2, 46.9)
- moved D22 114.5 mm to (168.8, 46.8)
- moved D23 113.8 mm to (173.3, 46.8)
- moved D24 113.3 mm to (178.0, 46.8)
- moved D21 113.2 mm to (159.8, 46.9)
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Connections:
- R10 pad 1: /A4 -> /S1
- R10 pad 2: Net-(D5-A) -> Net-(D10-A)
- R11 pad 1: /VCC -> /S2
- R11 pad 2: /A5 -> Net-(D11-A)
- R12 pad 1: /A5 -> /S3
- R12 pad 2: Net-(D6-A) -> Net-(D12-A)
- R13 pad 1: /VCC -> /S4
- R13 pad 2: /A6 -> Net-(D13-A)
- R14 pad 1: /A6 -> /S5
- R14 pad 2: Net-(D7-A) -> Net-(D14-A)
- R15 pad 1: /VCC -> /S6
- R15 pad 2: /A7 -> Net-(D15-A)
- R16 pad 1: /A7 -> /S7
- R16 pad 2: Net-(D8-A) -> Net-(D16-A)
- R17 pad 1: /VCC -> /A7
- R17 pad 2: /B0 -> Net-(D8-A)
- R18 pad 1: /B0 -> /A6
- R18 pad 2: Net-(D9-A) -> Net-(D7-A)
- R19 pad 1: /VCC -> /B1
- R19 pad 2: /B1 -> Net-(D19-A)
- R2 pad 1: /A0 -> /VCC
- R2 pad 2: Net-(D1-A) -> /A1
- R20 pad 1: /B1 -> /B2
- R20 pad 2: Net-(D10-A) -> Net-(D20-A)
- R21 pad 1: /VCC -> /A5
- R21 pad 2: /B2 -> Net-(D6-A)
- R22 pad 1: /B2 -> /A4
- R22 pad 2: Net-(D11-A) -> Net-(D5-A)
- R23 pad 1: /VCC -> /A3
- R23 pad 2: /B3 -> Net-(D4-A)
- R24 pad 1: /B3 -> /A2
- R24 pad 2: Net-(D12-A) -> Net-(D3-A)
- R25 pad 1: /VCC -> /A1
- R25 pad 2: /B4 -> Net-(D2-A)
- R26 pad 1: /B4 -> /A0
- R26 pad 2: Net-(D13-A) -> Net-(D1-A)
- R27 pad 2: /B5 -> /B0
- R28 pad 1: /B5 -> /B0
- R28 pad 2: Net-(D14-A) -> Net-(D18-A)
- R29 pad 2: /B6 -> /B1
- R3 pad 2: /A1 -> /A2
- R30 pad 1: /B6 -> /B3
- R30 pad 2: Net-(D15-A) -> Net-(D21-A)
- R31 pad 2: /B7 -> /B2
- R32 pad 1: /B7 -> /B4
- R32 pad 2: Net-(D16-A) -> Net-(D22-A)
- R33 pad 1: /S7 -> /VCC
- R33 pad 2: Net-(D17-A) -> /B3
- R34 pad 1: /S6 -> /B5
- R34 pad 2: Net-(D18-A) -> Net-(D23-A)
- R35 pad 1: /S5 -> /VCC
- R35 pad 2: Net-(D19-A) -> /B4
- R36 pad 1: /S4 -> /B6
- R36 pad 2: Net-(D20-A) -> Net-(D24-A)
- R37 pad 1: /S3 -> /VCC
- R37 pad 2: Net-(D21-A) -> /B5
- R38 pad 1: /S2 -> /B7
- R38 pad 2: Net-(D22-A) -> Net-(D25-A)
- R39 pad 1: /S1 -> /VCC
- R39 pad 2: Net-(D23-A) -> /B6
- R4 pad 1: /A1 -> /VCC
- R4 pad 2: Net-(D2-A) -> /A3
- R40 pad 1: /S0 -> /VCC
- R40 pad 2: Net-(D24-A) -> /B7
- R5 pad 2: /A2 -> /A4
- R6 pad 1: /A2 -> /VCC
- R6 pad 2: Net-(D3-A) -> /A5
- R7 pad 2: /A3 -> /A6
- R8 pad 1: /A3 -> /VCC
- R8 pad 2: Net-(D4-A) -> /A7
- R9 pad 1: /VCC -> /S0
- R9 pad 2: /A4 -> Net-(D9-A)
- SW1 pad 2: /A2 -> /A0
- SW10 pad 2: /B1 -> /A5
- SW11 pad 2: /B2 -> /A6
- SW12 pad 2: /B3 -> /A7
- SW2 pad 2: /A3 -> /A2
- SW3 pad 2: /A0 -> /A3
- SW4 pad 2: /A4 -> /B1
- SW6 pad 2: /A5 -> /B3
- SW7 pad 2: /A6 -> /B0
- SW8 pad 2: /A7 -> /B2
- SW9 pad 2: /B0 -> /A4
Routing:
- net GND: track 43.5 -> 802.8 mm, vias 0 -> 1
- net /B4: track 6.59 -> 295.6 mm, vias 0 -> 2
- net /A1: track 7.50 -> 255.0 mm, vias 0 -> 2
- net /A3: track 7.50 -> 240.3 mm, vias 0 -> 2
- net /VCC: track 43.4 -> 275.0 mm, vias 0 -> 2
- net /B7: track 6.59 -> 202.0 mm, vias 0 -> 1
- net /A0: track 8.92 -> 202.6 mm, vias 0 -> 2
- net /B5: track 6.59 -> 194.9 mm, vias 0 -> 2
- net /B6: track 6.59 -> 178.5 mm, vias 0 -> 2
- net /B0: track 6.13 -> 175.0 mm, vias 0 -> 1
- net /A6: track 7.50 -> 165.8 mm, vias 0 -> 1
- net /A2: track 7.50 -> 161.4 mm, vias 0 -> 1
- net /B3: track 6.42 -> 155.5 mm, vias 0 -> 2
- net /A7: track 7.62 -> 137.0 mm, vias 0 -> 1
- net /A4: track 7.50 -> 129.2 mm, vias 0 -> 1
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Other:
- board outline added: 249.5 x 146.8 mm

Commit message: commit
Other:
- board size 249.5 x 146.8 mm -> 255.5 x 159.5 mm
Changed lines of the file:
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@@
 		(embedded_fonts no)
 	)
+	(gr_circle
+		(center 259 169)
+		(end 262 169)
+		(stroke
+			(width 0.05)
+			(type solid)
+		)
+		(fill no)
+		(layer "Edge.Cuts")
+	)
+	(gr_circle
+		(center 15 21.5)
+		(end 18 21.5)
+		(stroke
+			(width 0.05)
+			(type solid)
+		)
+		(fill no)
+		(layer "Edge.Cuts")
+	)
+	(gr_circle
+		(center 15 171)
+		(end 18 171)
+		(stroke
+			(width 0.05)
+			(type solid)
+		)
+		(fill no)
+		(layer "Edge.Cuts")
+	)
 	(gr_rect
-		(start 16.25 16.5)
-		(end 265.75 163.25)
+		(start 10.25 16.5)
+		(end 265.75 176)
 		(stroke
 			(width 0.05)
@@
 		)
 		(fill no)
+		(layer "Edge.Cuts")
+	)
+	(gr_circle
+		(center 261 21.5)
+		(end 264 21.5)
+		(stroke
+			(width 0.05)
+			(type solid)
+		)
+		(fill no)
